File: can.brd (EAGLE design)
At the start: 55.2 x 35.5 mm, 36 parts, among them IC1 LM1117IMP-5.0, J1 AVR_SPI_PRG_6NS, Q1 FDS5680, Q2 FDS5680, Q3 FDS5680, U1 ATMEGA8, U2 MCP2510SO, U3 MCP2551SN, U5 SG-8002CA

Commit message: 1.0.2
Parts:
- removed C5, C6: (no value), SparkFun-Capacitors:1206
- removed U5: SG-8002CA, SparkFun-FreqCtrl:CRYSTAL-SMD-7X5
- removed Y2: (no value), SparkFun-FreqCtrl:HC49US
- added Y1, Y3: 16MHz, SparkFun-FreqCtrl:RESONATOR-SMD
- moved C1 20.1 mm to (19.1, 26.0), turned to 270 degrees
- moved LED4 9.67 mm to (29.8, 6.99), turned to 270 degrees
- moved R7 9.38 mm to (29.8, 11.4), turned to 270 degrees
- moved R8 6.63 mm to (32.4, 12.1), turned to 270 degrees
- moved LED2 6.48 mm to (32.4, 6.99), turned to 270 degrees
- moved IC1 1.91 mm to (10.2, 8.26)
Connections:
- removed net OSC1: C5.2, U1.7, U2.8, Y2.2
- removed net OSC2: C6.2, U1.8, U2.7, Y2.1
- new net N$12: U1.7, Y1.1
- new net N$14: U1.8, Y1.3
- new net N$16: U2.8, Y3.1
- new net N$19: U2.7, Y3.3
- net VSS: now also Y1.2, Y3.2; no longer C5.1, C6.1
Routing:
- net OSC1: track 18.9 -> 0.00 mm
- net OSC2: track 18.3 -> 0.00 mm
- net N$3: track 14.7 -> 3.85 mm
- net N$1: track 13.0 -> 5.72 mm
- net N$19: track 0.00 -> 4.60 mm
- net N$14: track 0.00 -> 4.35 mm
- net N$12: track 0.00 -> 4.24 mm
- net N$16: track 0.00 -> 3.76 mm
- net N$17: track 0.00 -> 2.68 mm
- net N$18: track 0.00 -> 2.04 mm
- net IN: track 12.8 -> 11.3 mm
- net VDD: track 68.2 -> 67.5 mm
