File: can.sch (EAGLE design)
At the start: 32 parts, among them J1 AVR_SPI_PRG_6NS, Q1 FDS5680, Q2 FDS5680, Q3 FDS5680, U1 ATMEGA8, U2 MCP2510SO, U3 MCP2551SN

Commit message: 1.0.0
Parts:
- removed C1, C2: (no value), SparkFun-Capacitors:CAP1206
- removed Y1: (no value), SparkFun-FreqCtrl:CRYSTALHC49US
- R6: device SparkFun-Passives:RESISTOR0805-RES -> SparkFun-Passives:RESISTOR1206
- R7, R8: device SparkFun-Resistors:RESISTOR1206 -> SparkFun-Resistors:RESISTOR0805-RES
Connections:
- removed net N$12: R8.1, U1.PD4(XCK/T0)
- removed net N$4: C1.2, U1.PB6(XTAL1/TOSC1), Y1.2
- removed net N$5: C2.2, U1.PB7(XTAL2/TOSC2), Y1.1
- removed net N$9: R7.1, U1.PD3(INT1)
- new net OSC1: C5.2, U1.PB6(XTAL1/TOSC1), U2>NAME.OSC1, Y2.2
- new net OSC2: C6.2, U1.PB7(XTAL2/TOSC2), U2>NAME.OSC2, Y2.1
- net CANH: now also JP4.2; no longer JP4.1
- net CANL: now also JP4.1; no longer JP4.2
- net N$1: now also R8.1, U1.PD6(AIN0); no longer C5.2, U2>NAME.OSC1, Y2.2
- net N$3: now also R7.1, U1.PD5(T1); no longer C6.2, U2>NAME.OSC2, Y2.1
- net RS: now also R5.2; no longer R5.1
- net VSS: now also R5.1; no longer C1.1, C2.1, R5.2
Other:
- moved on the sheet: C5, C6, LED2, LED4, R5, R7, R8, Y2
